Commit message: Descriptioniin oma robo. RViz toimii.

File: description/urdf/diffbot_description.urdf.xacro (robot description, xacro)
@@ -1,161 +1,77 @@
-<?xml version="1.0"?>
+<?xml version="1.0" ?>
 <robot xmlns:xacro="http://www.ros.org/wiki/xacro">
   <xacro:macro name="diffbot" params="prefix">
-  <!-- Constants for robot dimensions -->
-  <xacro:property name="PI" value="3.1415926535897931"/>
-  <xacro:property name="base_mass" value="0.3" /> <!-- arbitrary value for base mass -->
-  <xacro:property name="base_width" value="0.1" />
-  <xacro:property name="base_length" value="0.1" />
-  <xacro:property name="base_height" value="0.05" />
-  <xacro:property name="wheel_mass" value="0.3" /> <!-- arbitrary value for wheel mass -->
-  <xacro:property name="wheel_len" value="0.020" />
-  <xacro:property name="wheel_radius" value="0.015" />
-  <xacro:property name="caster_wheel_mass" value="0.1" /> <!-- arbitrary value for caster wheel mass -->
-  <xacro:property name="caster_wheel_radius" value="0.015" />
-  <xacro:property name="z_offset" value="-${base_height/2}" /> <!-- Space btw top of beam and the each joint -->
-  <!-- Base Link -->
   <link name="${prefix}base_link">
+    <inertial>
+      <origin xyz="0.18789605284929195 0.0 0.1382956611517429" rpy="0 0 0"/>
+      <mass value="36.30754966612175"/>
+      <inertia ixx="0.506671" iyy="1.080663" izz="1.439708" ixy="-0.0" iyz="0.0" ixz="0.031283"/>
+    </inertial>
+    <visual>
+      <origin xyz="0 0 0" rpy="0 0 0"/>
+      <geometry>
+        <mesh filename="package://hoverboard_driver/meshes/base_link.stl" scale="0.001 0.001 0.001"/>
+      </geometry>
+      <material name="red"/>
+    </visual>
     <collision>
       <origin xyz="0 0 0" rpy="0 0 0"/>
       <geometry>
-        <box size="${base_width} ${base_length} ${base_height}"/>
+        <mesh filename="package://hoverboard_driver/meshes/base_link.stl" scale="0.001 0.001 0.001"/>
       </geometry>
     </collision>
+  </link>
+  <link name="${prefix}right_wheel">
+    <inertial>
+      <origin xyz="-1.1074098332670195e-17 -0.02749999999999997 0.0" rpy="0 0 0"/>
+      <mass value="1.5275827380970637"/>
+      <inertia ixx="0.004015" iyy="0.007261" izz="0.004015" ixy="-0.0" iyz="0.0" ixz="-0.0"/>
+    </inertial>
     <visual>
-      <origin xyz="0 0 ${base_height/2}" rpy="0 0 0"/>
+      <origin xyz="-0.0 0.165 -0.0975" rpy="0 0 0"/>
       <geometry>
-        <box size="${base_width} ${base_length} ${base_height}"/>
+        <mesh filename="package://hoverboard_driver/meshes/right_wheel.stl" scale="0.001 0.001 0.001"/>
       </geometry>
-      <material name="orange"/>
+      <material name="black"/>
     </visual>
+    <collision>
+      <origin xyz="-0.0 0.165 -0.0975" rpy="0 0 0"/>
+      <geometry>
+        <mesh filename="package://hoverboard_driver/meshes/right_wheel.stl" scale="0.001 0.001 0.001"/>
+      </geometry>
+    </collision>
+  </link>
+  <link name="${prefix}left_wheel">
     <inertial>
-      <origin xyz="0 0 0" rpy="0 0 0"/>
-      <mass value="${base_mass}"/>
-      <inertia
-        ixx="${base_mass / 12.0 * (base_length*base_length + base_height*base_height)}" ixy="0.0" ixz="0.0"
-        iyy="${base_mass / 12.0 * (base_height*base_height + base_width*base_width)}" iyz="0.0"
-        izz="${base_mass / 12.0 * (base_width*base_width + base_length*base_length)}"/>
-      </inertial>
-    </link>
-    <joint name="${prefix}left_wheel_joint" type="continuous">
-      <parent link="${prefix}base_link"/>
-      <child link="${prefix}left_wheel"/>
-      <origin xyz="0 -${base_width/2} ${z_offset}" rpy="0 0 0"/>
-      <axis xyz="0 1 0"/>
-      <dynamics damping="0.2"/>
-    </joint>
-    <!-- left wheel Link -->
-    <link name="${prefix}left_wheel">
-      <collision>
-        <origin xyz="0 0 0" rpy="${PI/2} 0 0"/>
-        <geometry>
-          <cylinder length="${wheel_len}" radius="${wheel_radius}"/>
-        </geometry>
-      </collision>
-      <visual>
-        <origin xyz="0 0 0" rpy="${PI/2} 0 0"/>
-        <geometry>
-          <cylinder length="${wheel_len}" radius="${wheel_radius}"/>
-        </geometry>
-        <material name="black"/>
-      </visual>
-      <inertial>
-        <origin xyz="0 0 0" rpy="${PI/2} 0 0"/>
-        <mass value="${wheel_mass}"/>
-        <inertia
-          ixx="${wheel_mass / 12.0 * (3*wheel_radius*wheel_radius + wheel_len*wheel_len)}" ixy="0.0" ixz="0.0"
-          iyy="${wheel_mass / 12.0 * (3*wheel_radius*wheel_radius + wheel_len*wheel_len)}" iyz="0.0"
-          izz="${wheel_mass / 2.0 * wheel_radius*wheel_radius}"/>
-        </inertial>
-      </link>
-    <joint name="${prefix}right_wheel_joint" type="continuous">
-      <parent link="${prefix}base_link"/>
-      <child link="${prefix}right_wheel"/>
-      <origin xyz="0 ${base_width/2} ${z_offset}" rpy="0 0 0"/>
-      <axis xyz="0 1 0"/>
-      <dynamics damping="0.2"/>
-    </joint>
-    <!-- right wheel Link -->
-    <link name="${prefix}right_wheel">
-      <collision>
-        <origin xyz="0 0 0" rpy="${PI/2} 0 0"/>
-        <geometry>
-          <cylinder length="${wheel_len}" radius="${wheel_radius}"/>
-        </geometry>
-      </collision>
-      <visual>
-        <origin xyz="0 0 0" rpy="${PI/2} 0 0"/>
-        <geometry>
-          <cylinder length="${wheel_len}" radius="${wheel_radius}"/>
-        </geometry>
-        <material name="black"/>
-      </visual>
-      <inertial>
-        <origin xyz="0 0 0" rpy="${PI/2} 0 0"/>
-        <mass value="${wheel_mass}"/>
-        <inertia
-          ixx="${wheel_mass / 12.0 * (3*wheel_radius*wheel_radius + wheel_len*wheel_len)}" ixy="0.0" ixz="0.0"
-          iyy="${wheel_mass / 12.0 * (3*wheel_radius*wheel_radius + wheel_len*wheel_len)}" iyz="0.0"
-          izz="${wheel_mass / 2.0 * wheel_radius*wheel_radius}"/>
-        </inertial>
-      </link>
-    <joint name="${prefix}caster_frontal_wheel_joint" type="fixed">
-      <parent link="${prefix}base_link"/>
-      <child link="${prefix}caster_frontal_wheel"/>
-      <origin xyz="${base_width/2 - caster_wheel_radius} 0 ${z_offset}" rpy="0 0 0"/>
-    </joint>
-    <!-- caster frontal wheel Link -->
-    <link name="${prefix}caster_frontal_wheel">
-      <collision>
-        <origin xyz="0 0 0" rpy="0 0 0"/>
-        <geometry>
-          <sphere radius="${caster_wheel_radius}"/>
-        </geometry>
-      </collision>
-      <visual>
-        <origin xyz="0 0 0" rpy="0 0 0"/>
-        <geometry>
-          <sphere radius="${caster_wheel_radius}"/>
-        </geometry>
-        <material name="white"/>
-      </visual>
-      <inertial>
-        <origin xyz="0 0 0" rpy="0 0 0"/>
-        <mass value="${caster_wheel_mass}"/>
-        <inertia
-          ixx="${caster_wheel_mass * 0.4 * (caster_wheel_radius * caster_wheel_radius)}" ixy="0.0" ixz="0.0"
-          iyy="${caster_wheel_mass * 0.4 * (caster_wheel_radius * caster_wheel_radius)}" iyz="0.0"
-          izz="${caster_wheel_mass * 0.4 * (caster_wheel_radius * caster_wheel_radius)}"/>
-        </inertial>
-      </link>
-    <joint name="${prefix}caster_rear_wheel_joint" type="fixed">
-      <parent link="${prefix}base_link"/>
-      <child link="${prefix}caster_rear_wheel"/>
-      <origin xyz="${-base_width/2 + caster_wheel_radius} 0 ${z_offset}" rpy="0 0 0"/>
-    </joint>
-    <!-- caster rear wheel Link -->
-    <link name="${prefix}caster_rear_wheel">
-      <collision>
-        <origin xyz="0 0 0" rpy="0 0 0"/>
-        <geometry>
-          <sphere radius="${caster_wheel_radius}"/>
-        </geometry>
-      </collision>
-      <visual>
-        <origin xyz="0 0 0" rpy="0 0 0"/>
-        <geometry>
-          <sphere radius="${caster_wheel_radius}"/>
-        </geometry>
-        <material name="white"/>
-      </visual>
-      <inertial>
-        <origin xyz="0 0 0" rpy="0 0 0"/>
-        <mass value="${caster_wheel_mass}"/>
-        <inertia
-          ixx="${caster_wheel_mass * 0.4 * (caster_wheel_radius * caster_wheel_radius)}" ixy="0.0" ixz="0.0"
-          iyy="${caster_wheel_mass * 0.4 * (caster_wheel_radius * caster_wheel_radius)}" iyz="0.0"
-          izz="${caster_wheel_mass * 0.4 * (caster_wheel_radius * caster_wheel_radius)}"/>
-        </inertial>
-      </link>
+      <origin xyz="2.2148196665340383e-17 0.027499999999999997 1.3877787807814457e-17" rpy="0 0 0"/>
+      <mass value="1.5275827380970644"/>
+      <inertia ixx="0.004015" iyy="0.007261" izz="0.004015" ixy="0.0" iyz="0.0" ixz="0.0"/>
+    </inertial>
+    <visual>
+      <origin xyz="-0.0 -0.165 -0.0975" rpy="0 0 0"/>
+      <geometry>
+        <mesh filename="package://hoverboard_driver/meshes/left_wheel.stl" scale="0.001 0.001 0.001"/>
+      </geometry>
+      <material name="black"/>
+    </visual>
+    <collision>
+      <origin xyz="-0.0 -0.165 -0.0975" rpy="0 0 0"/>
+      <geometry>
+        <mesh filename="package://hoverboard_driver/meshes/left_wheel.stl" scale="0.001 0.001 0.001"/>
+      </geometry>
+    </collision>
+  </link>
+  <joint name="${prefix}right_wheel_joint" type="continuous">
+    <origin xyz="0.0 -0.165 0.0975" rpy="0 0 0"/>
+    <parent link="base_link"/>
+    <child link="right_wheel"/>
+    <axis xyz="0.0 -1.0 0.0"/>
+  </joint>
+  <joint name="${prefix}left_wheel_joint" type="continuous">
+    <origin xyz="0.0 0.165 0.0975" rpy="0 0 0"/>
+    <parent link="base_link"/>
+    <child link="left_wheel"/>
+    <axis xyz="0.0 1.0 0.0"/>
+  </joint>
   </xacro:macro>
 </robot>

Commit message: Lisätty urdf lidar ja kamera.

File: description/urdf/diffbot_description.urdf.xacro (robot description, xacro)
@@ -4,8 +4,8 @@
   <link name="${prefix}base_link">
     <inertial>
-      <origin xyz="0.18789605284929195 0.0 0.1382956611517429" rpy="0 0 0"/>
-      <mass value="36.30754966612175"/>
-      <inertia ixx="0.506671" iyy="1.080663" izz="1.439708" ixy="-0.0" iyz="0.0" ixz="0.031283"/>
-    </inertial>
+      <origin xyz="0.1868283906560058 -8.473062492372848e-18 0.13904584968795905" rpy="0 0 0"/>
+      <mass value="36.40957482835499"/>
+      <inertia ixx="0.50646" iyy="1.081484" izz="1.438296" ixy="-0.0" iyz="0.0" ixz="0.031938"/>
+  </inertial>
     <visual>
       <origin xyz="0 0 0" rpy="0 0 0"/>
@@ -24,8 +24,8 @@
   <link name="${prefix}right_wheel">
     <inertial>
-      <origin xyz="-1.1074098332670195e-17 -0.02749999999999997 0.0" rpy="0 0 0"/>
+      <origin xyz="0.0 -0.02749999999999997 0.0" rpy="0 0 0"/>
       <mass value="1.5275827380970637"/>
-      <inertia ixx="0.004015" iyy="0.007261" izz="0.004015" ixy="-0.0" iyz="0.0" ixz="-0.0"/>
-    </inertial>
+      <inertia ixx="0.004015" iyy="0.007261" izz="0.004015" ixy="0.0" iyz="0.0" ixz="0.0"/>
+  </inertial>
     <visual>
       <origin xyz="-0.0 0.165 -0.0975" rpy="0 0 0"/>
@@ -62,4 +62,85 @@
     </collision>
   </link>
+  <link name="${prefix}lidar">
+    <inertial>
+      <origin xyz="6.938893903907228e-18 0.0 0.007500000000000062" rpy="0 0 0"/>
+      <mass value="0.026012387171723484"/>
+      <inertia ixx="3e-06" iyy="3e-06" izz="5e-06" ixy="0.0" iyz="-0.0" ixz="0.0"/>
+    </inertial>
+    <visual>
+      <origin xyz="-0.051 -0.0 -0.2645" rpy="0 0 0"/>
+      <geometry>
+        <mesh filename="package://hoverboard_driver/meshes/lidar.stl" scale="0.001 0.001 0.001"/>
+      </geometry>
+      <material name="blue"/>
+    </visual>
+    <collision>
+      <origin xyz="-0.051 -0.0 -0.2645" rpy="0 0 0"/>
+      <geometry>
+        <mesh filename="package://hoverboard_driver/meshes/lidar.stl" scale="0.001 0.001 0.001"/>
+      </geometry>
+    </collision>
+  </link>
+  <link name="${prefix}camera">
+    <inertial>
+      <origin xyz="0.0030000000000000165 4.440892098500626e-18 -2.7755575615628914e-17" rpy="0 0 0"/>
+      <mass value="0.0051749999999999964"/>
+      <inertia ixx="1e-06" iyy="0.0" izz="0.0" ixy="0.0" iyz="-0.0" ixz="0.0"/>
+    </inertial>
+    <visual>
+      <origin xyz="-0.086 -0.0 -0.248" rpy="0 0 0"/>
+      <geometry>
+        <mesh filename="package://hoverboard_driver/meshes/camera.stl" scale="0.001 0.001 0.001"/>
+      </geometry>
+      <material name="blue"/>
+    </visual>
+    <collision>
+      <origin xyz="-0.086 -0.0 -0.248" rpy="0 0 0"/>
+      <geometry>
+        <mesh filename="package://hoverboard_driver/meshes/camera.stl" scale="0.001 0.001 0.001"/>
+      </geometry>
+    </collision>
+  </link>
+  <link name="${prefix}camera_optical"></link>
+  <link name="${prefix}caster_wheel_right">
+    <inertial>
+      <origin xyz="-3.4701079232313248e-09 -5.551115123125783e-17 -0.009375003732038686" rpy="0 0 0"/>
+      <mass value="0.030434215177785065"/>
+      <inertia ixx="5e-06" iyy="5e-06" izz="8e-06" ixy="-0.0" iyz="0.0" ixz="-0.0"/>
+    </inertial>
+    <visual>
+      <origin xyz="-0.41 0.136 -0.025" rpy="0 0 0"/>
+      <geometry>
+        <mesh filename="package://hoverboard_driver/meshes/caster_wheel_right.stl" scale="0.001 0.001 0.001"/>
+      </geometry>
+      <material name="black"/>
+    </visual>
+    <collision>
+      <origin xyz="-0.41 0.136 -0.025" rpy="0 0 0"/>
+      <geometry>
+        <mesh filename="package://hoverboard_driver/meshes/caster_wheel_right.stl" scale="0.001 0.001 0.001"/>
+      </geometry>
+    </collision>
+  </link>
+  <link name="${prefix}caster_wheel_left">
+    <inertial>
+      <origin xyz="-3.4701078122090223e-09 2.7755575615628914e-17 -0.009375000000000001" rpy="0 0 0"/>
+      <mass value="0.030434178831651098"/>
+      <inertia ixx="5e-06" iyy="5e-06" izz="8e-06" ixy="0.0" iyz="-0.0" ixz="-0.0"/>
+    </inertial>
+    <visual>
+      <origin xyz="-0.41 -0.136 -0.025" rpy="0 0 0"/>
+      <geometry>
+        <mesh filename="package://hoverboard_driver/meshes/caster_wheel_left.stl" scale="0.001 0.001 0.001"/>
+      </geometry>
+      <material name="black"/>
+    </visual>
+    <collision>
+      <origin xyz="-0.41 -0.136 -0.025" rpy="0 0 0"/>
+      <geometry>
+        <mesh filename="package://hoverboard_driver/meshes/caster_wheel_left.stl" scale="0.001 0.001 0.001"/>
+      </geometry>
+    </collision>
+  </link>
   <joint name="${prefix}right_wheel_joint" type="continuous">
     <origin xyz="0.0 -0.165 0.0975" rpy="0 0 0"/>
@@ -74,4 +155,29 @@
     <axis xyz="0.0 1.0 0.0"/>
   </joint>
+  <joint name="${prefix}lidar_joint" type="fixed">
+    <origin xyz="0.051 0.0 0.2645" rpy="0 0 0"/>
+    <parent link="base_link"/>
+    <child link="lidar"/>
+  </joint>
+  <joint name="${prefix}camera_joint" type="fixed">
+    <origin xyz="0.086 0.0 0.248" rpy="0 0 0"/>
+    <parent link="base_link"/>
+    <child link="camera"/>
+  </joint>
+  <joint name="${prefix}camera_optical_joint" type="fixed">
+    <origin xyz="0 0 0" rpy="${-pi/2} 0 ${-pi/2}"/>
+    <parent link="camera"/>
+    <child link="camera_optical"/>
+  </joint>
+  <joint name="${prefix}caster_wheel_right_joint" type="fixed">
+    <origin xyz="0.41 -0.136 0.025" rpy="0 0 0"/>
+    <parent link="base_link"/>
+    <child link="caster_wheel_right"/>
+  </joint>
+  <joint name="${prefix}caster_wheel_left_joint" type="fixed">
+    <origin xyz="0.41 0.136 0.025" rpy="0 0 0"/>
+    <parent link="base_link"/>
+    <child link="caster_wheel_left"/>
+  </joint>
   </xacro:macro>
 </robot>

Commit message: Lisätty IMU urdf. Ei vielä muuten käytössä.

File: description/urdf/diffbot_description.urdf.xacro (robot description, xacro)
@@ -143,4 +143,24 @@
     </collision>
   </link>
+  <link name="${prefix}imu_link">
+    <inertial>
+      <origin xyz="-1.8775462989895075e-09 0.0 0.0010000000000000009" rpy="0 0 0"/>
+      <mass value="0.009171939999999965"/>
+      <inertia ixx="0.0" iyy="0.0" izz="1e-06" ixy="0.0" iyz="0.0" ixz="-0.0"/>
+    </inertial>
+    <visual>
+      <origin xyz="-0.065 -0.0 -0.144" rpy="0 0 0"/>
+      <geometry>
+        <mesh filename="package://hoverboard_driver/meshes/imu_link.stl" scale="0.001 0.001 0.001"/>
+      </geometry>
+      <material name="blue"/>
+    </visual>
+    <collision>
+      <origin xyz="-0.065 -0.0 -0.144" rpy="0 0 0"/>
+      <geometry>
+        <mesh filename="package://hoverboard_driver/meshes/imu_link.stl" scale="0.001 0.001 0.001"/>
+      </geometry>
+    </collision>
+  </link>
   <joint name="${prefix}right_wheel_joint" type="continuous">
     <origin xyz="0.0 -0.165 0.0975" rpy="0 0 0"/>
@@ -180,4 +200,9 @@
     <child link="caster_wheel_left"/>
   </joint>
+  <joint name="${prefix}imu_joint" type="fixed">
+    <origin xyz="0.065 0.0 0.144" rpy="0 0 0"/>
+    <parent link="base_link"/>
+    <child link="imu_link"/>
+  </joint>
   </xacro:macro>
 </robot>

Commit message: SLAM mapping lisäyksiä (lidar)

File: description/urdf/diffbot_description.urdf.xacro (robot description, xacro)
@@ -205,4 +205,12 @@
     <child link="imu_link"/>
   </joint>
+<!-- BASE_FOOTPRINT -->
+    <joint name="${prefix}base_footprint_joint" type="fixed">
+        <parent link="base_link"/>
+        <child link="base_footprint"/>
+        <origin xyz="0 0 0" rpy="0 0 0"/>
+    </joint>
+    <link name="base_footprint">
+    </link>
   </xacro:macro>
 </robot>

Commit message: GPS URDF link ja joint

File: description/urdf/diffbot_description.urdf.xacro (robot description, xacro)
@@ -163,4 +163,24 @@
     </collision>
   </link>
+  <link name="${prefix}gps_link">
+    <inertial>
+      <origin xyz="4.619359950108759e-09 0.0 0.009999999999999981" rpy="0 0 0"/>
+      <mass value="0.09108000271439554"/>
+      <inertia ixx="3e-05" iyy="2.6e-05" izz="5e-05" ixy="-0.0" iyz="-0.0" ixz="0.0"/>
+    </inertial>
+    <visual>
+      <origin xyz="-0.31 -0.0 -0.165" rpy="0 0 0"/>
+      <geometry>
+        <mesh filename="package://hoverboard_driver/meshes/gps_link.stl" scale="0.001 0.001 0.001"/>
+      </geometry>
+      <material name="blue"/>
+    </visual>
+    <collision>
+      <origin xyz="-0.31 -0.0 -0.165" rpy="0 0 0"/>
+      <geometry>
+        <mesh filename="package://hoverboard_driver/meshes/gps_link.stl" scale="0.001 0.001 0.001"/>
+      </geometry>
+    </collision>
+  </link>
   <joint name="${prefix}right_wheel_joint" type="continuous">
     <origin xyz="0.0 -0.165 0.0975" rpy="0 0 0"/>
@@ -204,4 +224,9 @@
     <parent link="base_link"/>
     <child link="imu_link"/>
+  </joint>
+  <joint name="${prefix}gps_joint" type="fixed">
+    <origin xyz="0.31 0.0 0.165" rpy="0 0 0"/>
+    <parent link="base_link"/>
+    <child link="gps_link"/>
   </joint>
 <!-- BASE_FOOTPRINT -->

Commit message: EKA AUTOMAATTISESTI TOIMIVA BETA VERSIO 1.
Update configuration files and launch scripts for improved navigation and sensor integration

- Adjusted EKF parameters in ekf.yaml for better odometry configuration.
- Modified GPS parameters in gps.yaml to enhance measurement rates and output settings.
- Updated nav2_params.yaml to refine navigation behavior and goal checking mechanisms.
- Added new behavior tree for navigation to pose with improved goal checker integration.
- Introduced fusioncore.yaml for sensor fusion parameters and noise configurations. (FUSIONCORE EKA VERSIO, EI TOIMI)
- Created launch files for GPS and fusioncore nodes to streamline system startup. (FUSIONCORE EKA VERSIO, EI TOIMI)
- Enhanced arduino_bridge.py and joy_to_arduino.py for better command handling and state management.

File: description/urdf/diffbot_description.urdf.xacro (robot description, xacro)
@@ -238,4 +238,12 @@
     <link name="base_footprint">
     </link>
+<!-- gps -> gnss -->
+    <joint name="${prefix}gnss_joint" type="fixed">
+        <parent link="gps_link"/>
+        <child link="gnss_link"/>
+        <origin xyz="0 0 0" rpy="0 0 0"/>
+    </joint>
+    <link name="gnss_link">
+    </link>
   </xacro:macro>
 </robot>
