Commit message: URDF: right wheel joint axis +Y like the left (visual spin direction fix)
Since the Phase 2 driver sign fix both joint positions are positive when
driving forward (verified in-air: both wheels +27.93 rad after identical
forward drive). The old -Y axis was compensating the pre-rewrite driver's
inverted right-wheel position and made the right wheel render backwards
in Foxglove/RViz. Visualization-only: diff_drive never reads URDF axes.

Gotcha documented in the file: xacro comments must not contain colon+space,
the launch YAML-parses robot_description and fails on it.

Co-Authored-By: Claude Fable 5 <noreply@anthropic.com>

File: description/urdf/diffbot_description.urdf.xacro (robot description, xacro)
@@ -187,5 +187,10 @@
     <parent link="base_link"/>
     <child link="right_wheel"/>
-    <axis xyz="0.0 -1.0 0.0"/>
+    <!-- +Y like the left wheel. Since the Phase 2 driver sign fix both joint
+         positions are positive when driving forward; the old -Y flip was
+         compensating the driver's inverted right-wheel position.
+         NOTE - no colon characters in comments here, the launch file YAML-parses
+         the xacro output and a colon+space breaks robot_description. -->
+    <axis xyz="0.0 1.0 0.0"/>
   </joint>
   <joint name="${prefix}left_wheel_joint" type="continuous">
